File: midi_to_cv.sch (EAGLE design)
At the start: 32 parts, among them IC1 TL084P, U1 ATMEGA328P_PDIP

Commit message: converting to 4822
Parts:
- removed U$3: MCP4922-E/P, MCP4922:MCP4922-E/P
- added U$4, U$5: MCP4822-E/P, MCP4822:MCP4822-E/P
Connections:
- new net N$30: OK1.VO, R3.1
- net +5V: now also U$4.VDD; no longer U$3.VDD, U$3.VREFA, U$3.VREFB
- net GND: now also U$4.AVSS, U$4.~LDAC; no longer U$3.AVSS, U$3.~LDAC
- net N$10: no longer OK1.VO, R3.1
- net N$14: now also U$4.VOUTB; no longer U$3.VOUTB
- net N$2: now also U$4.VOUTA; no longer U$3.VOUTA
- net N$25: now also U$4.SCK; no longer U$3.SCK
- net N$26: now also U$4.SDI; no longer U$3.SDI
- net N$27: now also U$4.~CS; no longer U$3.~CS
Changed lines of the file:
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@@
 <part name="IC1" library="linear" deviceset="TL084" device="P"/>
 <part name="U$2" library="MCP4922" deviceset="MCP4922-E/P" device=""/>
-<part name="U$3" library="MCP4922" deviceset="MCP4922-E/P" device=""/>
 <part name="D1" library="diode" deviceset="1N4148" device="DO35-10"/>
 <part name="R2" library="rcl" deviceset="R-US_" device="0207/10" value="220"/>
@@
 <part name="GND8" library="supply1" deviceset="GND" device=""/>
 <part name="GND9" library="supply1" deviceset="GND" device=""/>
+<part name="U$4" library="MCP4822" deviceset="MCP4822-E/P" device=""/>
+<part name="U$5" library="MCP4822" deviceset="MCP4822-E/P" device=""/>
 </parts>
 <sheets>
@@
 <instance part="IC1" gate="D" x="149.86" y="22.86"/>
 <instance part="U$2" gate="A" x="106.68" y="50.8"/>
-<instance part="U$3" gate="A" x="106.68" y="114.3"/>
 <instance part="D1" gate="G$1" x="-22.86" y="114.3" rot="R90"/>
 <instance part="R2" gate="G$1" x="-33.02" y="119.38"/>
@@
 <instance part="GND8" gate="1" x="86.36" y="81.28"/>
 <instance part="GND9" gate="1" x="86.36" y="17.78"/>
+<instance part="U$4" gate="A" x="106.68" y="124.46"/>
+<instance part="U$5" gate="A" x="55.88" y="-12.7"/>
 </instances>
 <busses>
@@
 <net name="N$10" class="0">
 <segment>
-<pinref part="OK1" gate="G$1" pin="VO"/>
-<wire x1="10.16" y1="114.3" x2="15.24" y2="114.3" width="0.1524" layer="91"/>
-<wire x1="15.24" y1="114.3" x2="15.24" y2="111.76" width="0.1524" layer="91"/>
-<pinref part="R3" gate="G$1" pin="1"/>
-<wire x1="15.24" y1="111.76" x2="25.4" y2="111.76" width="0.1524" layer="91"/>
-<wire x1="25.4" y1="111.76" x2="25.4" y2="114.3" width="0.1524" layer="91"/>
 <pinref part="U1" gate="G$1" pin="PD0(RXD)"/>
 <wire x1="43.18" y1="50.8" x2="48.26" y2="50.8" width="0.1524" layer="91"/>
-<wire x1="48.26" y1="50.8" x2="48.26" y2="91.44" width="0.1524" layer="91"/>
-<wire x1="48.26" y1="91.44" x2="25.4" y2="91.44" width="0.1524" layer="91"/>
-<wire x1="25.4" y1="91.44" x2="25.4" y2="111.76" width="0.1524" layer="91"/>
-<junction x="25.4" y="111.76"/>
+<wire x1="48.26" y1="50.8" x2="48.26" y2="88.9" width="0.1524" layer="91"/>
 </segment>
 </net>
@@
 </segment>
 <segment>
-<pinref part="U$3" gate="A" pin="VDD"/>
 <pinref part="P+6" gate="1" pin="+5V"/>
-<wire x1="88.9" y1="129.54" x2="81.28" y2="129.54" width="0.1524" layer="91"/>
-<wire x1="81.28" y1="129.54" x2="81.28" y2="137.16" width="0.1524" layer="91"/>
 <pinref part="U$2" gate="A" pin="VDD"/>
 <wire x1="88.9" y1="66.04" x2="81.28" y2="66.04" width="0.1524" layer="91"/>
-<wire x1="81.28" y1="66.04" x2="81.28" y2="121.92" width="0.1524" layer="91"/>
-<junction x="81.28" y="129.54"/>
+<wire x1="81.28" y1="66.04" x2="81.28" y2="129.54" width="0.1524" layer="91"/>
 <pinref part="U$2" gate="A" pin="VREFA"/>
-<wire x1="81.28" y1="121.92" x2="81.28" y2="124.46" width="0.1524" layer="91"/>
-<wire x1="81.28" y1="124.46" x2="81.28" y2="129.54" width="0.1524" layer="91"/>
+<wire x1="81.28" y1="129.54" x2="81.28" y2="137.16" width="0.1524" layer="91"/>
 <wire x1="88.9" y1="60.96" x2="81.28" y2="60.96" width="0.1524" layer="91"/>
 <wire x1="81.28" y1="60.96" x2="81.28" y2="66.04" width="0.1524" layer="91"/>
@@
 <wire x1="81.28" y1="58.42" x2="81.28" y2="60.96" width="0.1524" layer="91"/>
 <junction x="81.28" y="60.96"/>
-<pinref part="U$3" gate="A" pin="VREFA"/>
-<wire x1="88.9" y1="124.46" x2="81.28" y2="124.46" width="0.1524" layer="91"/>
-<junction x="81.28" y="124.46"/>
-<pinref part="U$3" gate="A" pin="VREFB"/>
-<wire x1="88.9" y1="121.92" x2="81.28" y2="121.92" width="0.1524" layer="91"/>
-<junction x="81.28" y="121.92"/>
+<pinref part="U$4" gate="A" pin="VDD"/>
+<wire x1="88.9" y1="129.54" x2="81.28" y2="129.54" width="0.1524" layer="91"/>
+<junction x="81.28" y="129.54"/>
 </segment>
 </net>
@@
 </segment>
 <segment>
-<pinref part="U$3" gate="A" pin="~LDAC"/>
 <pinref part="GND8" gate="1" pin="GND"/>
-<wire x1="88.9" y1="109.22" x2="86.36" y2="109.22" width="0.1524" layer="91"/>
-<wire x1="86.36" y1="109.22" x2="86.36" y2="91.44" width="0.1524" layer="91"/>
-<wire x1="86.36" y1="91.44" x2="86.36" y2="83.82" width="0.1524" layer="91"/>
-<junction x="86.36" y="91.44"/>
-<pinref part="U$3" gate="A" pin="AVSS"/>
-<wire x1="88.9" y1="91.44" x2="86.36" y2="91.44" width="0.1524" layer="91"/>
+<wire x1="86.36" y1="116.84" x2="86.36" y2="111.76" width="0.1524" layer="91"/>
+<pinref part="U$4" gate="A" pin="~LDAC"/>
+<wire x1="86.36" y1="111.76" x2="86.36" y2="83.82" width="0.1524" layer="91"/>
+<wire x1="86.36" y1="116.84" x2="88.9" y2="116.84" width="0.1524" layer="91"/>
+<pinref part="U$4" gate="A" pin="AVSS"/>
+<wire x1="88.9" y1="111.76" x2="86.36" y2="111.76" width="0.1524" layer="91"/>
+<junction x="86.36" y="111.76"/>
 </segment>
 </net>
@@
 <net name="N$2" class="0">
 <segment>
-<pinref part="U$3" gate="A" pin="VOUTA"/>
 <pinref part="R5" gate="G$1" pin="1"/>
 <wire x1="124.46" y1="129.54" x2="127" y2="129.54" width="0.1524" layer="91"/>
+<pinref part="U$4" gate="A" pin="VOUTA"/>
 </segment>
 </net>
@@
 <net name="N$14" class="0">
 <segment>
-<pinref part="U$3" gate="A" pin="VOUTB"/>
 <wire x1="124.46" y1="127" x2="127" y2="127" width="0.1524" layer="91"/>
 <wire x1="127" y1="127" x2="127" y2="99.06" width="0.1524" layer="91"/>
 <pinref part="R10" gate="G$1" pin="1"/>
 <wire x1="127" y1="99.06" x2="137.16" y2="99.06" width="0.1524" layer="91"/>
+<pinref part="U$4" gate="A" pin="VOUTB"/>
 </segment>
 </net>
@@
 <pinref part="U1" gate="G$1" pin="PB2(SS/OC1B)"/>
 <wire x1="43.18" y1="22.86" x2="63.5" y2="22.86" width="0.1524" layer="91"/>
-<wire x1="63.5" y1="22.86" x2="63.5" y2="114.3" width="0.1524" layer="91"/>
-<pinref part="U$3" gate="A" pin="SCK"/>
-<wire x1="63.5" y1="114.3" x2="88.9" y2="114.3" width="0.1524" layer="91"/>
+<wire x1="63.5" y1="22.86" x2="63.5" y2="121.92" width="0.1524" layer="91"/>
+<pinref part="U$4" gate="A" pin="SCK"/>
+<wire x1="63.5" y1="121.92" x2="88.9" y2="121.92" width="0.1524" layer="91"/>
 </segment>
 </net>
@@
 <pinref part="U1" gate="G$1" pin="PB3(MOSI/OC2)"/>
 <wire x1="43.18" y1="20.32" x2="66.04" y2="20.32" width="0.1524" layer="91"/>
-<wire x1="66.04" y1="20.32" x2="66.04" y2="111.76" width="0.1524" layer="91"/>
-<pinref part="U$3" gate="A" pin="SDI"/>
-<wire x1="66.04" y1="111.76" x2="88.9" y2="111.76" width="0.1524" layer="91"/>
+<wire x1="66.04" y1="20.32" x2="66.04" y2="119.38" width="0.1524" layer="91"/>
+<pinref part="U$4" gate="A" pin="SDI"/>
+<wire x1="66.04" y1="119.38" x2="88.9" y2="119.38" width="0.1524" layer="91"/>
 </segment>
 </net>
@@
 <pinref part="U1" gate="G$1" pin="PB4(MISO)"/>
 <wire x1="43.18" y1="17.78" x2="68.58" y2="17.78" width="0.1524" layer="91"/>
-<wire x1="68.58" y1="17.78" x2="68.58" y2="116.84" width="0.1524" layer="91"/>
-<pinref part="U$3" gate="A" pin="~CS"/>
-<wire x1="68.58" y1="116.84" x2="88.9" y2="116.84" width="0.1524" layer="91"/>
+<wire x1="68.58" y1="17.78" x2="68.58" y2="124.46" width="0.1524" layer="91"/>
+<pinref part="U$4" gate="A" pin="~CS"/>
+<wire x1="68.58" y1="124.46" x2="88.9" y2="124.46" width="0.1524" layer="91"/>
 </segment>
 </net>
@@
 </segment>
 </net>
+<net name="N$30" class="0">
+<segment>
+<pinref part="R3" gate="G$1" pin="1"/>
+<pinref part="OK1" gate="G$1" pin="VO"/>
+<wire x1="10.16" y1="114.3" x2="15.24" y2="114.3" width="0.1524" layer="91"/>
+<wire x1="15.24" y1="114.3" x2="15.24" y2="111.76" width="0.1524" layer="91"/>
+<wire x1="15.24" y1="111.76" x2="25.4" y2="111.76" width="0.1524" layer="91"/>
+<wire x1="25.4" y1="111.76" x2="25.4" y2="114.3" width="0.1524" layer="91"/>
+<junction x="25.4" y="111.76"/>
+<wire x1="25.4" y1="88.9" x2="25.4" y2="111.76" width="0.1524" layer="91"/>
+</segment>
+</net>

Commit message: converted to 4822
Parts:
- removed U$2: MCP4922-E/P, MCP4922:MCP4922-E/P
Connections:
- removed net N$10: U1.PD0(RXD)
- net +5V: now also U$5.VDD; no longer U$2.VDD, U$2.VREFA, U$2.VREFB
- net GND: now also U$5.AVSS, U$5.~LDAC; no longer U$2.AVSS, U$2.~LDAC
- net N$18: now also U$5.VOUTA; no longer U$2.VOUTA
- net N$23: now also U$5.SDI; no longer U$2.SDI
- net N$24: now also U$5.VOUTB; no longer U$2.VOUTB
- net N$28: now also U$5.SCK; no longer U$2.SCK
- net N$29: now also U$5.~CS; no longer U$2.~CS
- net N$30: now also U1.PD0(RXD)
Other:
- moved on the sheet: U$5
Changed lines of the file:
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@@
 <part name="C3" library="rcl" deviceset="C-US" device="025-040X050" value=".1uF"/>
 <part name="IC1" library="linear" deviceset="TL084" device="P"/>
-<part name="U$2" library="MCP4922" deviceset="MCP4922-E/P" device=""/>
 <part name="D1" library="diode" deviceset="1N4148" device="DO35-10"/>
 <part name="R2" library="rcl" deviceset="R-US_" device="0207/10" value="220"/>
@@
 <part name="PAD6" library="wirepad" deviceset="2,54/0,9" device="" value="mod output"/>
 <part name="P+6" library="supply1" deviceset="+5V" device=""/>
-<part name="GND8" library="supply1" deviceset="GND" device=""/>
-<part name="GND9" library="supply1" deviceset="GND" device=""/>
 <part name="U$4" library="MCP4822" deviceset="MCP4822-E/P" device=""/>
 <part name="U$5" library="MCP4822" deviceset="MCP4822-E/P" device=""/>
+<part name="GND10" library="supply1" deviceset="GND" device=""/>
 </parts>
 <sheets>
@@
 <instance part="IC1" gate="C" x="149.86" y="63.5"/>
 <instance part="IC1" gate="D" x="149.86" y="22.86"/>
-<instance part="U$2" gate="A" x="106.68" y="50.8"/>
 <instance part="D1" gate="G$1" x="-22.86" y="114.3" rot="R90"/>
 <instance part="R2" gate="G$1" x="-33.02" y="119.38"/>
@@
 <instance part="PAD6" gate="1" x="172.72" y="22.86" rot="MR0"/>
 <instance part="P+6" gate="1" x="81.28" y="139.7"/>
-<instance part="GND8" gate="1" x="86.36" y="81.28"/>
-<instance part="GND9" gate="1" x="86.36" y="17.78"/>
 <instance part="U$4" gate="A" x="106.68" y="124.46"/>
-<instance part="U$5" gate="A" x="55.88" y="-12.7"/>
+<instance part="U$5" gate="A" x="106.68" y="60.96"/>
+<instance part="GND10" gate="1" x="86.36" y="38.1"/>
 </instances>
 <busses>
@@
 <pinref part="R2" gate="G$1" pin="1"/>
 <wire x1="-45.72" y1="119.38" x2="-38.1" y2="119.38" width="0.1524" layer="91"/>
-</segment>
-</net>
-<net name="N$10" class="0">
-<segment>
-<pinref part="U1" gate="G$1" pin="PD0(RXD)"/>
-<wire x1="43.18" y1="50.8" x2="48.26" y2="50.8" width="0.1524" layer="91"/>
-<wire x1="48.26" y1="50.8" x2="48.26" y2="88.9" width="0.1524" layer="91"/>
 </segment>
 </net>
@@
 <segment>
 <pinref part="P+6" gate="1" pin="+5V"/>
-<pinref part="U$2" gate="A" pin="VDD"/>
+<wire x1="81.28" y1="129.54" x2="81.28" y2="137.16" width="0.1524" layer="91"/>
+<pinref part="U$4" gate="A" pin="VDD"/>
+<wire x1="88.9" y1="129.54" x2="81.28" y2="129.54" width="0.1524" layer="91"/>
+<pinref part="U$5" gate="A" pin="VDD"/>
 <wire x1="88.9" y1="66.04" x2="81.28" y2="66.04" width="0.1524" layer="91"/>
 <wire x1="81.28" y1="66.04" x2="81.28" y2="129.54" width="0.1524" layer="91"/>
-<pinref part="U$2" gate="A" pin="VREFA"/>
-<wire x1="81.28" y1="129.54" x2="81.28" y2="137.16" width="0.1524" layer="91"/>
-<wire x1="88.9" y1="60.96" x2="81.28" y2="60.96" width="0.1524" layer="91"/>
-<wire x1="81.28" y1="60.96" x2="81.28" y2="66.04" width="0.1524" layer="91"/>
-<junction x="81.28" y="66.04"/>
-<pinref part="U$2" gate="A" pin="VREFB"/>
-<wire x1="88.9" y1="58.42" x2="81.28" y2="58.42" width="0.1524" layer="91"/>
-<wire x1="81.28" y1="58.42" x2="81.28" y2="60.96" width="0.1524" layer="91"/>
-<junction x="81.28" y="60.96"/>
-<pinref part="U$4" gate="A" pin="VDD"/>
-<wire x1="88.9" y1="129.54" x2="81.28" y2="129.54" width="0.1524" layer="91"/>
 <junction x="81.28" y="129.54"/>
 </segment>
@@
 </segment>
 <segment>
-<pinref part="R9" gate="G$1" pin="A"/>
-<pinref part="GND5" gate="1" pin="GND"/>
-<wire x1="132.08" y1="76.2" x2="132.08" y2="73.66" width="0.1524" layer="91"/>
-</segment>
-<segment>
 <pinref part="GND6" gate="1" pin="GND"/>
 <pinref part="R13" gate="G$1" pin="1"/>
@@
 </segment>
 <segment>
-<pinref part="U$2" gate="A" pin="~LDAC"/>
-<pinref part="GND9" gate="1" pin="GND"/>
-<wire x1="88.9" y1="45.72" x2="86.36" y2="45.72" width="0.1524" layer="91"/>
-<wire x1="86.36" y1="45.72" x2="86.36" y2="27.94" width="0.1524" layer="91"/>
-<pinref part="U$2" gate="A" pin="AVSS"/>
-<wire x1="86.36" y1="27.94" x2="86.36" y2="20.32" width="0.1524" layer="91"/>
-<wire x1="88.9" y1="27.94" x2="86.36" y2="27.94" width="0.1524" layer="91"/>
-<junction x="86.36" y="27.94"/>
-</segment>
-<segment>
-<pinref part="GND8" gate="1" pin="GND"/>
+<pinref part="U$5" gate="A" pin="AVSS"/>
+<pinref part="GND10" gate="1" pin="GND"/>
+<wire x1="88.9" y1="48.26" x2="86.36" y2="48.26" width="0.1524" layer="91"/>
+<wire x1="86.36" y1="48.26" x2="86.36" y2="40.64" width="0.1524" layer="91"/>
+<pinref part="U$5" gate="A" pin="~LDAC"/>
+<wire x1="88.9" y1="53.34" x2="86.36" y2="53.34" width="0.1524" layer="91"/>
+<wire x1="86.36" y1="53.34" x2="86.36" y2="48.26" width="0.1524" layer="91"/>
+<junction x="86.36" y="48.26"/>
 <wire x1="86.36" y1="116.84" x2="86.36" y2="111.76" width="0.1524" layer="91"/>
 <pinref part="U$4" gate="A" pin="~LDAC"/>
-<wire x1="86.36" y1="111.76" x2="86.36" y2="83.82" width="0.1524" layer="91"/>
 <wire x1="86.36" y1="116.84" x2="88.9" y2="116.84" width="0.1524" layer="91"/>
 <pinref part="U$4" gate="A" pin="AVSS"/>
 <wire x1="88.9" y1="111.76" x2="86.36" y2="111.76" width="0.1524" layer="91"/>
 <junction x="86.36" y="111.76"/>
+<wire x1="86.36" y1="111.76" x2="86.36" y2="53.34" width="0.1524" layer="91"/>
+<junction x="86.36" y="53.34"/>
+</segment>
+<segment>
+<pinref part="R9" gate="G$1" pin="A"/>
+<pinref part="GND5" gate="1" pin="GND"/>
+<wire x1="132.08" y1="76.2" x2="132.08" y2="73.66" width="0.1524" layer="91"/>
 </segment>
 </net>
@@
 <wire x1="172.72" y1="83.82" x2="172.72" y2="96.52" width="0.1524" layer="91"/>
 <junction x="172.72" y="96.52"/>
-</segment>
-</net>
-<net name="N$18" class="0">
-<segment>
-<pinref part="U$2" gate="A" pin="VOUTA"/>
-<pinref part="IC1" gate="C" pin="+IN"/>
-<wire x1="124.46" y1="66.04" x2="142.24" y2="66.04" width="0.1524" layer="91"/>
 </segment>
 </net>
@@
 <net name="N$24" class="0">
 <segment>
-<pinref part="U$2" gate="A" pin="VOUTB"/>
+<pinref part="IC1" gate="D" pin="+IN"/>
+<wire x1="127" y1="25.4" x2="142.24" y2="25.4" width="0.1524" layer="91"/>
+<pinref part="U$5" gate="A" pin="VOUTB"/>
 <wire x1="124.46" y1="63.5" x2="127" y2="63.5" width="0.1524" layer="91"/>
 <wire x1="127" y1="63.5" x2="127" y2="25.4" width="0.1524" layer="91"/>
-<pinref part="IC1" gate="D" pin="+IN"/>
-<wire x1="127" y1="25.4" x2="142.24" y2="25.4" width="0.1524" layer="91"/>
 </segment>
 </net>
@@
 <pinref part="U1" gate="G$1" pin="PD7(AIN1)"/>
 <wire x1="43.18" y1="33.02" x2="71.12" y2="33.02" width="0.1524" layer="91"/>
-<wire x1="71.12" y1="33.02" x2="71.12" y2="50.8" width="0.1524" layer="91"/>
-<pinref part="U$2" gate="A" pin="SCK"/>
-<wire x1="88.9" y1="50.8" x2="71.12" y2="50.8" width="0.1524" layer="91"/>
+<wire x1="71.12" y1="33.02" x2="71.12" y2="58.42" width="0.1524" layer="91"/>
+<pinref part="U$5" gate="A" pin="SCK"/>
+<wire x1="71.12" y1="58.42" x2="88.9" y2="58.42" width="0.1524" layer="91"/>
 </segment>
 </net>
@@
 <pinref part="U1" gate="G$1" pin="PB0(ICP)"/>
 <wire x1="43.18" y1="27.94" x2="73.66" y2="27.94" width="0.1524" layer="91"/>
-<wire x1="73.66" y1="27.94" x2="73.66" y2="48.26" width="0.1524" layer="91"/>
-<pinref part="U$2" gate="A" pin="SDI"/>
-<wire x1="73.66" y1="48.26" x2="88.9" y2="48.26" width="0.1524" layer="91"/>
+<wire x1="73.66" y1="27.94" x2="73.66" y2="55.88" width="0.1524" layer="91"/>
+<pinref part="U$5" gate="A" pin="SDI"/>
+<wire x1="73.66" y1="55.88" x2="88.9" y2="55.88" width="0.1524" layer="91"/>
 </segment>
 </net>
@@
 <pinref part="U1" gate="G$1" pin="PB1(OC1A)"/>
 <wire x1="43.18" y1="25.4" x2="76.2" y2="25.4" width="0.1524" layer="91"/>
-<wire x1="76.2" y1="25.4" x2="76.2" y2="53.34" width="0.1524" layer="91"/>
-<pinref part="U$2" gate="A" pin="~CS"/>
-<wire x1="76.2" y1="53.34" x2="88.9" y2="53.34" width="0.1524" layer="91"/>
+<wire x1="76.2" y1="25.4" x2="76.2" y2="60.96" width="0.1524" layer="91"/>
+<pinref part="U$5" gate="A" pin="~CS"/>
+<wire x1="76.2" y1="60.96" x2="88.9" y2="60.96" width="0.1524" layer="91"/>
 </segment>
 </net>
@@
 <junction x="25.4" y="111.76"/>
 <wire x1="25.4" y1="88.9" x2="25.4" y2="111.76" width="0.1524" layer="91"/>
-</segment>
-</net>
+<pinref part="U1" gate="G$1" pin="PD0(RXD)"/>
+<wire x1="43.18" y1="50.8" x2="48.26" y2="50.8" width="0.1524" layer="91"/>
+<wire x1="48.26" y1="50.8" x2="48.26" y2="88.9" width="0.1524" layer="91"/>
+<wire x1="25.4" y1="88.9" x2="48.26" y2="88.9" width="0.1524" layer="91"/>
+</segment>
+</net>
+<net name="N$18" class="0">
+<segment>
+<pinref part="U$5" gate="A" pin="VOUTA"/>
+<pinref part="IC1" gate="C" pin="+IN"/>
+<wire x1="124.46" y1="66.04" x2="142.24" y2="66.04" width="0.1524" layer="91"/>
+</segment>
+</net>

Commit message: remembering the gate output
Parts:
- added PAD7: gate output, wirepad:2,54/0,9
Connections:
- new net N$10: PAD7.P, U1.PB5(SCK)
Changed lines of the file:
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@@
 <part name="U$5" library="MCP4822" deviceset="MCP4822-E/P" device=""/>
 <part name="GND10" library="supply1" deviceset="GND" device=""/>
+<part name="PAD7" library="wirepad" deviceset="2,54/0,9" device="" value="gate output"/>
 </parts>
 <sheets>
@@
 <instance part="U$5" gate="A" x="106.68" y="60.96"/>
 <instance part="GND10" gate="1" x="86.36" y="38.1"/>
+<instance part="PAD7" gate="1" x="55.88" y="5.08" rot="MR0"/>
 </instances>
 <busses>
@@
 </segment>
 </net>
+<net name="N$10" class="0">
+<segment>
+<pinref part="U1" gate="G$1" pin="PB5(SCK)"/>
+<wire x1="43.18" y1="15.24" x2="45.72" y2="15.24" width="0.1524" layer="91"/>
+<wire x1="45.72" y1="15.24" x2="45.72" y2="5.08" width="0.1524" layer="91"/>
+<pinref part="PAD7" gate="1" pin="P"/>
+<wire x1="45.72" y1="5.08" x2="53.34" y2="5.08" width="0.1524" layer="91"/>
+</segment>
+</net>
